Commit message: add camera urdf

File: kcare_description/robots/slamware.urdf.xacro (robot description, xacro)
@@ -4,4 +4,5 @@
   <xacro:property name="mesh_path" value="package://${package_name}/meshes"/>
   <xacro:include filename="$(find kcare_description)/robots/common/link.xacro"/> -->
+  <xacro:property name="mesh_path" value="package://kcare_description/meshes/"/>
   <xacro:common_link
     name="slam_base"
@@ -9,5 +10,5 @@
     mass="42.44816908546966"
     ixx="1.368829" iyy="1.544543" izz="1.587721" ixy="0.00047" iyz="0.00375" ixz="-0.000201"
-    mesh_file="${mesh_path}/slamware/base_link.stl"
+    mesh_file="${mesh_path}slamware/base_link.stl"
   />
   <xacro:common_link
@@ -16,5 +17,5 @@
     mass="3.867230"
     ixx="0.016843" iyy="0.009476" izz="0.009476" ixy="-0.000000" iyz="0.000000" ixz="0.000000"
-    mesh_file="${mesh_path}/slamware/slam_wheel.stl"
+    mesh_file="${mesh_path}slamware/slam_wheel.stl"
     material="black"
   />
@@ -24,5 +25,5 @@
     mass="3.867230"
     ixx="0.016843" iyy="0.009476" izz="0.009476" ixy="-0.000000" iyz="0.000000" ixz="0.000000"
-    mesh_file="${mesh_path}/slamware/slam_wheel.stl"
+    mesh_file="${mesh_path}slamware/slam_wheel.stl"
     material="black"
   />
@@ -32,5 +33,5 @@
     mass="1.177702"
     ixx="0.001147" iyy="0.001298" izz="0.000735" ixy="-0.000001" iyz="-0.000002" ixz="-0.000319"
-    mesh_file="${mesh_path}/slamware/caster.stl"
+    mesh_file="${mesh_path}slamware/caster.stl"
     material="black"
   />
@@ -40,5 +41,5 @@
     mass="1.177702"
     ixx="0.001147" iyy="0.001298" izz="0.000735" ixy="-0.000001" iyz="-0.000002" ixz="-0.000319"
-    mesh_file="${mesh_path}/slamware/caster.stl"
+    mesh_file="${mesh_path}slamware/caster.stl"
     material="black"
   />
@@ -48,5 +49,5 @@
     mass="1.177702"
     ixx="0.001147" iyy="0.001298" izz="0.000735" ixy="-0.000001" iyz="-0.000002" ixz="-0.000319"
-    mesh_file="${mesh_path}/slamware/caster.stl"
+    mesh_file="${mesh_path}slamware/caster.stl"
     material="black"
   />
@@ -56,5 +57,5 @@
     mass="1.177702"
     ixx="0.001147" iyy="0.001298" izz="0.000735" ixy="-0.000001" iyz="-0.000002" ixz="-0.000319"
-    mesh_file="${mesh_path}/slamware/caster.stl"
+    mesh_file="${mesh_path}slamware/caster.stl"
     material="black"
   />
