Commit message: Update URDF with clober

File: kcare_description/robots/_test_.urdf.xacro (robot description, xacro)
@@ -1,6 +1,13 @@
 <?xml version="1.0" ?>
 <robot name="kcare" xmlns:xacro="http://www.ros.org/wiki/xacro">
+  <!-- <xacro:include filename="$(find kcare_description)/robots/common/link.xacro"/>
+  <xacro:include filename="$(find former_description)/urdf/robot.urdf.xacro"/>
+  <xacro:include filename="$(find kcare_description)/robots/elevation.urdf.xacro"/>
+  <joint name="slam_to_elev_fix_joint" type="fixed">
+    <origin xyz="0.051 0.0 306.0e-3" rpy="0 0 0"/>
+    <parent link="base_footprint"/>
+    <child link="elevation_base"/>
+  </joint> -->
   <xacro:include filename="$(find kcare_description)/robots/common/link.xacro"/>
-  <xacro:include filename="$(find kcare_description)/robots/pan_tilt.urdf.xacro"/>
-  <!-- <xacro:include filename="$(find kcare_description)/robots/elevation.urdf.xacro"/> -->
+  <xacro:include filename="$(find kcare_description)/robots/clo_elevation.urdf.xacro"/>
 </robot>

File: kcare_description/robots/clo_elevation.urdf.xacro (robot description, xacro)
@@ -4,5 +4,5 @@
   <xacro:common_link
     name="elevation_base"
-    mesh_file="${mesh_path}elevation/elevation_base.stl"
+    mesh_file="${mesh_path}elevation/clo_elevation_base.stl"
   />
   <xacro:common_link
@@ -27,5 +27,5 @@
   </joint>
   <joint name="elevation_to_head_fix_joint" type="fixed">
-    <origin xyz="0.0 0.0 0.859" rpy="0 0 0"/>
+    <origin xyz="0.0 0.0 1.068" rpy="0 0 0"/>
     <parent link="elevation_base"/>
     <child link="head_base"/>

File: kcare_description/robots/common/link.xacro (robot description, xacro)
@@ -10,5 +10,5 @@
   mesh_file
   scale:='0.001 0.001 0.001'
-  material:='silver'">
+  material:='kcare_silver'">
   <!-- <xacro:macro name="common_link" params="name inertial_origin mass ixx iyy izz ixy iyz ixz mesh_file scale:='0.001 0.001 0.001' material:=silver"> -->
     <link name="${name}">

File: kcare_description/robots/common/materials.xacro (robot description, xacro)
@@ -1,8 +1,8 @@
 <?xml version="1.0" ?>
 <robot name="kcare" xmlns:xacro="http://www.ros.org/wiki/xacro">
-<material name="silver">
+<material name="kcare_silver">
   <color rgba="0.700 0.700 0.700 1.000"/>
 </material>
-<material name="black">
+<material name="kcare_black">
     <color rgba="0.2 0.2 0.2 1"/>
 </material>

File: kcare_description/robots/pan_tilt.urdf.xacro (robot description, xacro)
@@ -22,5 +22,5 @@
   <xacro:include filename="$(find kcare_description)/robots/femto_bolt.urdf.xacro"/>
   <joint name="pantilt_fix_joint" type="fixed">
-    <origin xyz="-0.094838 0.0 0.077" rpy="0 0 0"/>
+    <origin xyz="-0.055 0.0 0.077" rpy="0 0 0"/>
     <parent link="head_base"/>
     <child link="head_link1"/>

File: kcare_description/robots/slamware.urdf.xacro (robot description, xacro)
@@ -9,35 +9,35 @@
     name="left_wheel"
     mesh_file="${mesh_path}slamware/slam_wheel.stl"
-    material="black"
+    material="kcare_black"
   />
   <xacro:common_link
     name="right_wheel"
     mesh_file="${mesh_path}slamware/slam_wheel.stl"
-    material="black"
+    material="kcare_black"
   />
   <xacro:common_link
     name="lf_caster"
     mesh_file="${mesh_path}slamware/caster.stl"
-    material="black"
+    material="kcare_black"
   />
   <xacro:common_link
     name="rf_caster"
      mesh_file="${mesh_path}slamware/caster.stl"
-    material="black"
+    material="kcare_black"
   />
   <xacro:common_link
     name="lb_caster"
     mesh_file="${mesh_path}slamware/caster.stl"
-    material="black"
+    material="kcare_black"
   />
   <xacro:common_link
     name="rb_caster"
     mesh_file="${mesh_path}slamware/caster.stl"
-    material="black"
+    material="kcare_black"
   />
   <link name="elevation_base">
   </link>
   <joint name="left_wheel_joint" type="continuous">
-    <origin xyz="0.0 0.16885 0.0" rpy="0 0 -1.5708"/>
+    <origin xyz="0.0 0.16885 0.0" rpy="0 0 ${-90 * pi/180}"/>
     <parent link="slam_base"/>
     <child link="left_wheel"/>
@@ -45,5 +45,5 @@
   </joint>
   <joint name="right_wheel_joint" type="continuous">
-    <origin xyz="0.0 -0.16885 0.0" rpy="0 0 1.5708"/>
+    <origin xyz="0.0 -0.16885 0.0" rpy="0 0 ${90 * pi/180}"/>
     <parent link="slam_base"/>
     <child link="right_wheel"/>
@@ -71,5 +71,5 @@
   </joint>
   <joint name="slam_to_elev_fix_joint" type="fixed">
-    <origin xyz="0.0 0.0 0.362985" rpy="0 0 0"/>
+    <origin xyz="-0.04998 0.0 0.362985" rpy="0 0 0"/>
     <parent link="slam_base"/>
     <child link="elevation_base"/>

Commit message: hand urdf updating

File: kcare_description/robots/_test_.urdf.xacro (robot description, xacro)
@@ -1,13 +1,6 @@
 <?xml version="1.0" ?>
 <robot name="kcare" xmlns:xacro="http://www.ros.org/wiki/xacro">
-  <!-- <xacro:include filename="$(find kcare_description)/robots/common/link.xacro"/>
-  <xacro:include filename="$(find former_description)/urdf/robot.urdf.xacro"/>
-  <xacro:include filename="$(find kcare_description)/robots/elevation.urdf.xacro"/>
-  <joint name="slam_to_elev_fix_joint" type="fixed">
-    <origin xyz="0.051 0.0 306.0e-3" rpy="0 0 0"/>
-    <parent link="base_footprint"/>
-    <child link="elevation_base"/>
-  </joint> -->
+  <!-- <xacro:include filename="$(find kcare_description)/robots/device_d405.urdf.xacro"/> -->
   <xacro:include filename="$(find kcare_description)/robots/common/link.xacro"/>
-  <xacro:include filename="$(find kcare_description)/robots/clo_elevation.urdf.xacro"/>
+  <xacro:include filename="$(find kcare_description)/robots/hand_camera.urdf.xacro"/>
 </robot>
