Commit message: Update 250910

File: kcare_description/robots/clo_elevation.urdf.xacro (robot description, xacro)
@@ -22,5 +22,5 @@
   </joint>
   <joint name="elevation_to_arm_fix_joint" type="fixed">
-    <origin xyz="0.2415 0.0 0.0" rpy="0 0 ${-90 * pi/180}"/>
+    <origin xyz="0.2415 0.0 0.0" rpy="0 0 0"/>
     <parent link="linear_block"/>
     <child link="world"/>

File: kcare_description/robots/elevation.urdf.xacro (robot description, xacro)
@@ -22,5 +22,5 @@
   </joint>
   <joint name="elevation_to_arm_fix_joint" type="fixed">
-    <origin xyz="0.2415 0.0 0.0" rpy="0 0 ${-90 * pi/180}"/>
+    <origin xyz="0.2415 0.0 0.0" rpy="0 0 0"/>
     <parent link="linear_block"/>
     <child link="world"/>

File: kcare_description/robots/xarm7.urdf.xacro (robot description, xacro)
@@ -4,5 +4,5 @@
   <xacro:xarm_device
       dof="7"
-      add_gripper="true"
+      add_gripper="false"
   />
 </robot>
