Commit message: Update URDF

File: kcare_description/robots/common/link.xacro (robot description, xacro)
@@ -2,5 +2,14 @@
 <robot name="kcare" xmlns:xacro="http://www.ros.org/wiki/xacro">
   <xacro:include filename="$(find kcare_description)/robots/common/materials.xacro"/>
-  <xacro:macro name="common_link" params="name inertial_origin mass ixx iyy izz ixy iyz ixz mesh_file scale:='0.001 0.001 0.001' material:=silver">
+<xacro:macro name="common_link" params="
+  name
+  inertial_origin:='0 0 0'
+  mass:='0.5'
+  ixx:='0.002' iyy:='0.002' izz:='0.002'
+  ixy:='0.0' iyz:='0.0' ixz:='0.0'
+  mesh_file
+  scale:='0.001 0.001 0.001'
+  material:='silver'">
+  <!-- <xacro:macro name="common_link" params="name inertial_origin mass ixx iyy izz ixy iyz ixz mesh_file scale:='0.001 0.001 0.001' material:=silver"> -->
     <link name="${name}">
       <inertial>

File: kcare_description/robots/device_elevation.urdf.xacro (robot description, xacro)
@@ -2,5 +2,4 @@
 <robot name="kcare" xmlns:xacro="http://www.ros.org/wiki/xacro">
   <xacro:include filename="$(find kcare_description)/robots/common/link.xacro"/>
-  <xacro:include filename="$(find kcare_description)/robots/pan_tilt.urdf.xacro"/>
-  <!-- <xacro:include filename="$(find kcare_description)/robots/elevation.urdf.xacro"/> -->
+  <xacro:include filename="$(find kcare_description)/robots/elevation.urdf.xacro"/>
 </robot>

File: kcare_description/robots/device_head.urdf.xacro (robot description, xacro)
@@ -3,4 +3,3 @@
   <xacro:include filename="$(find kcare_description)/robots/common/link.xacro"/>
   <xacro:include filename="$(find kcare_description)/robots/pan_tilt.urdf.xacro"/>
-  <!-- <xacro:include filename="$(find kcare_description)/robots/elevation.urdf.xacro"/> -->
 </robot>

File: kcare_description/robots/kcare_platform.urdf.xacro (robot description, xacro)
@@ -53,5 +53,5 @@
     <child link="linear_block"/>
     <axis xyz="0.0 0.0 1.0"/>
-    <limit upper="0.68" lower="0.1" effort="100" velocity="100"/>
+    <limit upper="0.8" lower="0.0" effort="100" velocity="100"/>
   </joint>
   <joint name="lm_to_arm" type="fixed">

File: kcare_description/robots/slamware.urdf.xacro (robot description, xacro)
@@ -1,20 +1,11 @@
 <?xml version="1.0" ?>
 <robot name="slamtec" xmlns:xacro="http://www.ros.org/wiki/xacro">
-  <!-- <xacro:property name="package_name" value="kcare_description"/>
-  <xacro:property name="mesh_path" value="package://${package_name}/meshes"/>
-  <xacro:include filename="$(find kcare_description)/robots/common/link.xacro"/> -->
   <xacro:property name="mesh_path" value="package://kcare_description/meshes/"/>
   <xacro:common_link
     name="slam_base"
-    inertial_origin="-0.004242067006968334 0.0005565721742923574 0.176282566938588"
-    mass="42.44816908546966"
-    ixx="1.368829" iyy="1.544543" izz="1.587721" ixy="0.00047" iyz="0.00375" ixz="-0.000201"
     mesh_file="${mesh_path}slamware/base_link.stl"
   />
   <xacro:common_link
     name="left_wheel"
-    inertial_origin="-0.001865 0.052015 -0.010160"
-    mass="3.867230"
-    ixx="0.016843" iyy="0.009476" izz="0.009476" ixy="-0.000000" iyz="0.000000" ixz="0.000000"
     mesh_file="${mesh_path}slamware/slam_wheel.stl"
     material="black"
@@ -22,7 +13,4 @@
   <xacro:common_link
     name="right_wheel"
-    inertial_origin="-0.001865 0.052015 -0.010160"
-    mass="3.867230"
-    ixx="0.016843" iyy="0.009476" izz="0.009476" ixy="-0.000000" iyz="0.000000" ixz="0.000000"
     mesh_file="${mesh_path}slamware/slam_wheel.stl"
     material="black"
@@ -30,7 +18,4 @@
   <xacro:common_link
     name="lf_caster"
-    inertial_origin="-0.018022 -0.000120 -0.048838"
-    mass="1.177702"
-    ixx="0.001147" iyy="0.001298" izz="0.000735" ixy="-0.000001" iyz="-0.000002" ixz="-0.000319"
     mesh_file="${mesh_path}slamware/caster.stl"
     material="black"
@@ -38,15 +23,9 @@
   <xacro:common_link
     name="rf_caster"
-    inertial_origin="-0.018022 -0.000120 -0.048838"
-    mass="1.177702"
-    ixx="0.001147" iyy="0.001298" izz="0.000735" ixy="-0.000001" iyz="-0.000002" ixz="-0.000319"
-    mesh_file="${mesh_path}slamware/caster.stl"
+     mesh_file="${mesh_path}slamware/caster.stl"
     material="black"
   />
   <xacro:common_link
     name="lb_caster"
-    inertial_origin="-0.018022 -0.000120 -0.048838"
-    mass="1.177702"
-    ixx="0.001147" iyy="0.001298" izz="0.000735" ixy="-0.000001" iyz="-0.000002" ixz="-0.000319"
     mesh_file="${mesh_path}slamware/caster.stl"
     material="black"
@@ -54,10 +33,9 @@
   <xacro:common_link
     name="rb_caster"
-    inertial_origin="-0.018022 -0.000120 -0.048838"
-    mass="1.177702"
-    ixx="0.001147" iyy="0.001298" izz="0.000735" ixy="-0.000001" iyz="-0.000002" ixz="-0.000319"
     mesh_file="${mesh_path}slamware/caster.stl"
     material="black"
   />
+  <link name="elevation_base">
+  </link>
   <joint name="left_wheel_joint" type="continuous">
     <origin xyz="0.0 0.16885 0.0" rpy="0 0 -1.5708"/>
@@ -92,3 +70,8 @@
     <child link="rb_caster"/>
   </joint>
+  <joint name="slam_to_elev_fix_joint" type="fixed">
+    <origin xyz="0.0 0.0 0.362985" rpy="0 0 0"/>
+    <parent link="slam_base"/>
+    <child link="elevation_base"/>
+  </joint>
 </robot>

File: kcare_description/robots/xarm7.urdf.xacro (robot description, xacro)
@@ -1,11 +1,7 @@
 <?xml version="1.0" ?>
 <robot name="kcare" xmlns:xacro="http://www.ros.org/wiki/xacro">
-  <link name="arm_base"/>
   <xacro:include filename="$(find xarm_description)/urdf/xarm_device_macro.xacro" />
   <xacro:xarm_device
       dof="7"
-      attach_to="arm_base"
-      attach_xyz="0.0 0.0 0.0"
-      attach_rpy="0 0 0"
       add_gripper="true"
   />
